File: schema dmp/schema dmp.kicad_sch (KiCad schematic)
At the start: 36 parts, among them J1 +12v, J10 FAN2-, J2 GND, J3 +12v 2, J4 GND2, J5 out+ regulated, J6 out-, J7 FAN1+, J8 FAN1-, J9 FAN2+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

Commit message: added dps doc
Parts:
- added F1: Fuse 230V/16A, symbol Device:Fuse
- added J11: IEC320 L, symbol Connector:Conn_01x01_Pin
- added J12: IEC320 PE, symbol Connector:Conn_01x01_Pin
- added J13: IEC320 N, symbol Connector:Conn_01x01_Pin
- added J14: GND OUT, symbol Connector:Conn_01x01_Pin
- added PS1, PS2: VTX-214-015-112, symbol Converter_ACDC:VTX-214-015-112
Connections:
- new net: J13.1 (Pin_1), PS1.2 (N), PS2.2 (N)
- new net: F1.2, PS1.3 (L), PS2.3 (L)
- new net: F1.1, J11.1 (Pin_1)
- new net GNDREF: J12.1 (Pin_1), J14.1 (Pin_1)
- no-connect marks 1 -> 2
Other:
- moved on the sheet: A1, C1, C2, C3, D1, E1, E2, IO14, IO7, J10, J5, J6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
